File: Akashi-18.kicad_sch (KiCad schematic)
At the start: 8 parts, among them Q1 DTC143Z, Q2 DTC143Z, Q3 DTC143Z, U1 Pico

Commit message: Layout done
Parts:
- added RV1: RK09D117000B, Potentiometer_THT:Potentiometer_Alps_RK09K_Single_Vertical, symbol Device:R_Potentiometer_MountingPin
- added SW1, SW2, SW3: B3FS, Button_Switch_THT:SW_TH_Tactile_Omron_B3F-10xx, symbol Switch:SW_Omron_B3FS
- D1: footprint (none) -> LED_THT:LED_D5.0mm-4_RGB
- Q1, Q2, Q3: footprint (none) -> Package_TO_SOT_THT:TO-92_Inline
- R1, R2, R3: footprint (none) -> Resistor_THT:R_Axial_DIN0207_L6.3mm_D2.5mm_P10.16mm_Horizontal
- U1: footprint RPi_Pico:RPi_Pico_SMD_TH -> Rpi_Pico:RPi_Pico_SMD_TH
Connections:
- net BLUE: now also Q3.3 (B), U1.29 (GPIO22); no longer Q3.1 (B), U1.6 (GPIO4)
- net GND: now also Q1.1 (E), Q2.1 (E), Q3.1 (E), U1.13 (GND), U1.18 (GND), U1.23 (GND), U1.28 (GND), U1.3 (GND), U1.33 (AGND), U1.38 (GND), U1.8 (GND), RV1.1, RV1.MP (MountPin), SW1.1, SW2.1, SW3.1; no longer Q1.2 (E), Q2.2 (E), Q3.2 (E)
- net GREEN: now also Q2.3 (B), U1.27 (GPIO21); no longer Q2.1 (B), U1.5 (GPIO3)
- net RED: now also Q1.3 (B), U1.26 (GPIO20); no longer Q1.1 (B), U1.4 (GPIO2)
- net at U1.14 (GPIO10): now also SW1.2
- net at U1.15 (GPIO11): now also SW2.2
- net at U1.16 (GPIO12): now also SW3.2
- net at U1.31 (GPIO26_ADC0): now also RV1.2
- net 3V3: now reaches U1.36 (3V3)
- net 3V3: now also RV1.3
- net at R2.2: now also Q2.2 (C); no longer Q2.3 (C)
- net at R3.2: now also Q3.2 (C); no longer Q3.3 (C)
- net at R1.2: now also Q1.2 (C); no longer Q1.3 (C)
- no-connect marks 0 -> 26
Other:
- moved on the sheet: D1, Q1, R1, R2, R3, U1

Commit message: All modified parts are registered to the local lib.
Parts:
- removed D1: OSTAMA5B31A, LED_THT:LED_D5.0mm-4_RGB, symbol Device:LED_GBAR
- removed Q1, Q2, Q3: DTC143Z, Package_TO_SOT_THT:TO-92_Inline, symbol Transistor_BJT:DTC143Z
- removed U1: Pico, Rpi_Pico:RPi_Pico_SMD_TH, symbol Rpi_Pico:Pico
- added D1: OSTAMA5B31A, My_Lib:LED_D5.0mm-4_RGB, symbol My_LED:LED_GBAR
- added Q1, Q2, Q3: DTC143Z, Package_TO_SOT_THT:TO-92_Inline, symbol My_Digital_Tr:DTC143Z_1
- added U1: Pico, My_Lib:RPi_Pico_SMD_TH, symbol My_RPi_Pico:Pico
Connections:
- net +5V: now also D1.3 (A), U1.40 (VBUS)
- net 3V3: now also U1.36 (3V3)
- net BLUE: now also Q3.3 (B), U1.29 (GPIO22)
- net GND: now also Q1.1 (E), Q2.1 (E), Q3.1 (E), U1.13 (GND), U1.18 (GND), U1.23 (GND), U1.28 (GND), U1.3 (GND), U1.33 (AGND), U1.38 (GND), U1.8 (GND)
- net GREEN: now also Q2.3 (B), U1.27 (GPIO21)
- net RED: now also Q1.3 (B), U1.26 (GPIO20)
- net at R2.2: now also Q2.2 (C)
- net at SW1.2: now also U1.15 (GPIO11)
- net at SW2.2: now also U1.16 (GPIO12)
- net at SW3.2: now also U1.17 (GPIO13)
- net at RV1.2: now also U1.31 (GPIO26_ADC0)
- net at R2.1: now also D1.1 (GK)
- net at R3.1: now also D1.2 (BK)
- net at R3.2: now also Q3.2 (C)
- net at R1.1: now also D1.4 (RK)
- net at R1.2: now also Q1.2 (C)

Commit message: Adjust the space of transistor.
Parts:
- R1: value R -> 220
- R2: value R -> 180
- R3: value R -> 91
Changed lines of the file:
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@@
       (effects (font (size 1.27 1.27)) (justify left))
     )
-    (property "Value" "R" (at 90.17 58.42 0)
+    (property "Value" "180" (at 90.17 58.42 0)
       (effects (font (size 1.27 1.27)) (justify left))
     )
@@
       (effects (font (size 1.27 1.27)) (justify left))
     )
-    (property "Value" "R" (at 102.87 58.42 0)
+    (property "Value" "91" (at 102.87 58.42 0)
       (effects (font (size 1.27 1.27)) (justify left))
     )
@@
       (effects (font (size 1.27 1.27)) (justify left))
     )
-    (property "Value" "R" (at 77.47 58.42 0)
-      (effects (font (size 1.27 1.27)) (justify left))
-    )
+    (property "Value" "220" (at 77.47 58.42 0)
+      (effects (font (size 1.27 1.27)) (justify left))
+    )

Commit message: Add capacitor
For RF Immunity reduction.
Also added parts list.
Parts:
- added C1: 0.1u, Capacitor_THT:C_Disc_D8.0mm_W2.5mm_P5.00mm, symbol Device:C
- R1: value 220 -> 150
- R2: value 180 -> 240
Connections:
- net GND: now also C1.2
- net at RV1.2, U1.31 (GPIO26_ADC0): now also C1.1
Other:
- moved on the sheet: RV1
Changed lines of the file:
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@@
   (junction (at 179.07 92.71) (diameter 0) (color 0 0 0 0)
   )
-  (junction (at 196.85 102.87) (diameter 0) (color 0 0 0 0)
+  (junction (at 207.01 102.87) (diameter 0) (color 0 0 0 0)
   )
   (junction (at 179.07 105.41) (diameter 0) (color 0 0 0 0)
   )
   (junction (at 133.35 105.41) (diameter 0) (color 0 0 0 0)
+  )
+  (junction (at 198.12 97.79) (diameter 0) (color 0 0 0 0)
   )
   (no_connect (at 138.43 120.65))
@@
     (stroke (width 0) (type default))
   )
+  (wire (pts (xy 198.12 97.79) (xy 198.12 99.06))
+    (stroke (width 0) (type default))
+  )
+  (wire (pts (xy 198.12 97.79) (xy 203.2 97.79))
+    (stroke (width 0) (type default))
+  )
   (wire (pts (xy 133.35 142.24) (xy 133.35 118.11))
     (stroke (width 0) (type default))
@@
     (stroke (width 0) (type default))
   )
-  (wire (pts (xy 173.99 85.09) (xy 196.85 85.09))
-    (stroke (width 0) (type default))
-  )
   (wire (pts (xy 87.63 72.39) (xy 87.63 60.96))
     (stroke (width 0) (type default))
@@
     (stroke (width 0) (type default))
   )
+  (wire (pts (xy 173.99 85.09) (xy 207.01 85.09))
+    (stroke (width 0) (type default))
+  )
   (wire (pts (xy 179.07 148.59) (xy 179.07 118.11))
     (stroke (width 0) (type default))
@@
     (stroke (width 0) (type default))
   )
-  (wire (pts (xy 196.85 85.09) (xy 196.85 93.98))
+  (wire (pts (xy 173.99 97.79) (xy 198.12 97.79))
+    (stroke (width 0) (type default))
+  )
+  (wire (pts (xy 207.01 85.09) (xy 207.01 93.98))
     (stroke (width 0) (type default))
   )
@@
     (stroke (width 0) (type default))
   )
-  (wire (pts (xy 196.85 102.87) (xy 203.2 102.87))
+  (wire (pts (xy 207.01 102.87) (xy 213.36 102.87))
     (stroke (width 0) (type default))
   )
@@
     (stroke (width 0) (type default))
   )
-  (wire (pts (xy 196.85 102.87) (xy 196.85 106.68))
+  (wire (pts (xy 207.01 102.87) (xy 207.01 106.68))
     (stroke (width 0) (type default))
   )
@@
     (stroke (width 0) (type default))
   )
-  (wire (pts (xy 196.85 101.6) (xy 196.85 102.87))
+  (wire (pts (xy 207.01 101.6) (xy 207.01 102.87))
     (stroke (width 0) (type default))
   )
@@
     (stroke (width 0) (type default))
   )
-  (wire (pts (xy 201.93 97.79) (xy 203.2 97.79))
-    (stroke (width 0) (type default))
-  )
-  (wire (pts (xy 173.99 97.79) (xy 193.04 97.79))
+  (wire (pts (xy 212.09 97.79) (xy 213.36 97.79))
     (stroke (width 0) (type default))
   )
@@
     (stroke (width 0) (type default))
   )
+  (wire (pts (xy 198.12 106.68) (xy 198.12 107.95))
+    (stroke (width 0) (type default))
+  )
   (wire (pts (xy 74.93 52.07) (xy 82.55 52.07))
     (stroke (width 0) (type default))
@@
     (stroke (width 0) (type default))
   )
-  (wire (pts (xy 203.2 97.79) (xy 203.2 102.87))
+  (wire (pts (xy 213.36 97.79) (xy 213.36 102.87))
     (stroke (width 0) (type default))
   )
@@
     (effects (font (size 1.27 1.27)) (justify left bottom))
   )
-  (label "3V3" (at 189.23 85.09 0) (fields_autoplaced)
+  (label "3V3" (at 199.39 85.09 0) (fields_autoplaced)
     (effects (font (size 1.27 1.27)) (justify left bottom))
   )
@@
       (effects (font (size 1.27 1.27)) (justify left))
     )
-    (property "Value" "180" (at 90.17 58.42 0)
+    (property "Value" "240" (at 90.17 58.42 0)
       (effects (font (size 1.27 1.27)) (justify left))
     )
@@
     )
   )
-  (symbol (lib_id "Device:R_Potentiometer_MountingPin") (at 196.85 97.79 180) (unit 1)
-    (in_bom yes) (on_board yes) (dnp no) (fields_autoplaced)
-    (property "Reference" "RV1" (at 214.63 92.8369 0)
-      (effects (font (size 1.27 1.27)))
-    )
-    (property "Value" "RK09D117000B" (at 214.63 95.3769 0)
-      (effects (font (size 1.27 1.27)))
-    )
-    (property "Footprint" "Potentiometer_THT:Potentiometer_Alps_RK09K_Single_Vertical" (at 196.85 97.79 0)
-      (effects (font (size 1.27 1.27)) hide)
-    )
-    (property "Datasheet" "~" (at 196.85 97.79 0)
+  (symbol (lib_id "Device:R_Potentiometer_MountingPin") (at 207.01 97.79 180) (unit 1)
+    (in_bom yes) (on_board yes) (dnp no) (fields_autoplaced)
+    (property "Reference" "RV1" (at 224.79 92.8369 0)
+      (effects (font (size 1.27 1.27)))
+    )
+    (property "Value" "RK09D117000B" (at 224.79 95.3769 0)
+      (effects (font (size 1.27 1.27)))
+    )
+    (property "Footprint" "Potentiometer_THT:Potentiometer_Alps_RK09K_Single_Vertical" (at 207.01 97.79 0)
+      (effects (font (size 1.27 1.27)) hide)
+    )
+    (property "Datasheet" "~" (at 207.01 97.79 0)
       (effects (font (size 1.27 1.27)) hide)
     )
@@
       (effects (font (size 1.27 1.27)) (justify left))
     )
-    (property "Value" "220" (at 77.47 58.42 0)
+    (property "Value" "150" (at 77.47 58.42 0)
       (effects (font (size 1.27 1.27)) (justify left))
     )
@@
     )
   )
-  (symbol (lib_id "power:GND") (at 196.85 106.68 0) (unit 1)
-    (in_bom yes) (on_board yes) (dnp no) (fields_autoplaced)
-    (property "Reference" "#PWR011" (at 196.85 113.03 0)
-      (effects (font (size 1.27 1.27)) hide)
-    )
-    (property "Value" "GND" (at 196.85 111.76 0)
-      (effects (font (size 1.27 1.27)))
-    )
-    (property "Footprint" "" (at 196.85 106.68 0)
-      (effects (font (size 1.27 1.27)) hide)
-    )
-    (property "Datasheet" "" (at 196.85 106.68 0)
+  (symbol (lib_id "power:GND") (at 207.01 106.68 0) (unit 1)
+    (in_bom yes) (on_board yes) (dnp no) (fields_autoplaced)
+    (property "Reference" "#PWR011" (at 207.01 113.03 0)
+      (effects (font (size 1.27 1.27)) hide)
+    )
+    (property "Value" "GND" (at 207.01 111.76 0)
+      (effects (font (size 1.27 1.27)))
+    )
+    (property "Footprint" "" (at 207.01 106.68 0)
+      (effects (font (size 1.27 1.27)) hide)
+    )
+    (property "Datasheet" "" (at 207.01 106.68 0)
       (effects (font (size 1.27 1.27)) hide)
     )
@@
     )
   )
+  (symbol (lib_id "Device:C") (at 198.12 102.87 0) (unit 1)
+    (in_bom yes) (on_board yes) (dnp no) (fields_autoplaced)
+    (property "Reference" "C1" (at 201.93 101.6 0)
+      (effects (font (size 1.27 1.27)) (justify left))
+    )
+    (property "Value" "0.1u" (at 201.93 104.14 0)
+      (effects (font (size 1.27 1.27)) (justify left))
+    )
+    (property "Footprint" "Capacitor_THT:C_Disc_D8.0mm_W2.5mm_P5.00mm" (at 199.0852 106.68 0)
+      (effects (font (size 1.27 1.27)) hide)
+    )
+    (property "Datasheet" "~" (at 198.12 102.87 0)
+      (effects (font (size 1.27 1.27)) hide)
+    )
+    (pin "1")
+    (pin "2")
+    (instances
+      (project "Akashi-18"
+        (path "/61a99dab-c882-441e-a650-f04a0666c89d"
+          (reference "C1") (unit 1)
+        )
+      )
+    )
+  )
   (symbol (lib_id "power:GND") (at 100.33 97.79 0) (unit 1)
     (in_bom yes) (on_board yes) (dnp no) (fields_autoplaced)
@@
         )
       )
+    )
+  )
+  (symbol (lib_id "power:GND") (at 198.12 107.95 0) (unit 1)
+    (in_bom yes) (on_board yes) (dnp no) (fields_autoplaced)
+    (property "Reference" "#PWR012" (at 198.12 114.3 0)
+      (effects (font (size 1.27 1.27)) hide)
+    )
+    (property "Value" "GND" (at 198.12 113.03 0)
+      (effects (font (size 1.27 1.27)))
+    )
+    (property "Footprint" "" (at 198.12 107.95 0)
+      (effects (font (size 1.27 1.27)) hide)
+    )
+    (property "Datasheet" "" (at 198.12 107.95 0)
+      (effects (font (size 1.27 1.27)) hide)
+    )
+    (pin "1")
+    (instances
+      (project "Akashi-18"
+        (path "/61a99dab-c882-441e-a650-f04a0666c89d"
+          (reference "#PWR012") (unit 1)
+        )
+      )

Commit message: Correct the parts list and refine the PCB layout.
Volume -> A-curve.
RasPi Pico -> wo Header.
Connector -> Conthrough.

PCB layout has been refined for the better visibility of the
RV1 comment.
Parts:
- RV1: value RK09D117000B -> RK09D117000C
Changed lines of the file:
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@@
   (symbol (lib_id "Device:R_Potentiometer_MountingPin") (at 207.01 97.79 180) (unit 1)
     (in_bom yes) (on_board yes) (dnp no) (fields_autoplaced)
-    (property "Reference" "RV1" (at 224.79 92.8369 0)
+    (property "Reference" "RV1" (at 218.44 92.8369 0)
       (effects (font (size 1.27 1.27)))
     )
-    (property "Value" "RK09D117000B" (at 224.79 95.3769 0)
+    (property "Value" "RK09D117000C" (at 218.44 95.3769 0)
       (effects (font (size 1.27 1.27)))
     )

Commit message: Update README.
Added Schematics PDF.
Other:
- title: (none) -> Pico Trainer
Changed lines of the file:
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@@
 (kicad_sch (version 20230121) (generator eeschema)
   (paper "A4")
+  (title_block
+    (title "Pico Trainer")
+    (date "2023-12-23")
+    (rev "1.0.0")
+  )
   (junction (at 133.35 142.24) (diameter 0) (color 0 0 0 0)
   )

Commit message: Change resitor value to good for the education.
- Update parts list.
- Added assembled board photo.
Parts:
- R1: value 150 -> 1.5k
- R2: value 240 -> 2.7k
- R3: value 91 -> 1k
Changed lines of the file:
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@@
       (effects (font (size 1.27 1.27)) (justify left))
     )
-    (property "Value" "240" (at 90.17 58.42 0)
+    (property "Value" "2.7k" (at 90.17 58.42 0)
       (effects (font (size 1.27 1.27)) (justify left))
     )
@@
       (effects (font (size 1.27 1.27)) (justify left))
     )
-    (property "Value" "91" (at 102.87 58.42 0)
+    (property "Value" "1k" (at 102.87 58.42 0)
       (effects (font (size 1.27 1.27)) (justify left))
     )
@@
       (effects (font (size 1.27 1.27)) (justify left))
     )
-    (property "Value" "150" (at 77.47 58.42 0)
-      (effects (font (size 1.27 1.27)) (justify left))
-    )
+    (property "Value" "1.5k" (at 77.47 58.42 0)
+      (effects (font (size 1.27 1.27)) (justify left))
+    )

Commit message: Add reset switch.
Parts:
- added SW4: B3FS, Button_Switch_THT:SW_TH_Tactile_Omron_B3F-10xx, symbol Switch:SW_Omron_B3FS
Connections:
- net GND: now also SW4.1
- net RESET: now reaches U1.30 (RUN)
- net RESET: now also SW4.2
- no-connect marks 26 -> 25
Changed lines of the file:
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@@
   (no_connect (at 173.99 113.03))
   (no_connect (at 173.99 90.17))
-  (no_connect (at 173.99 100.33))
   (no_connect (at 158.75 128.27))
   (no_connect (at 173.99 77.47))
@@
     (stroke (width 0) (type default))
   )
+  (wire (pts (xy 236.22 115.57) (xy 236.22 134.62))
+    (stroke (width 0) (type default))
+  )
   (wire (pts (xy 87.63 72.39) (xy 87.63 60.96))
     (stroke (width 0) (type default))
@@
     (stroke (width 0) (type default))
   )
+  (wire (pts (xy 236.22 144.78) (xy 236.22 148.59))
+    (stroke (width 0) (type default))
+  )
   (wire (pts (xy 124.46 142.24) (xy 133.35 142.24))
     (stroke (width 0) (type default))
@@
     (stroke (width 0) (type default))
   )
+  (wire (pts (xy 173.99 100.33) (xy 189.23 100.33))
+    (stroke (width 0) (type default))
+  )
   (wire (pts (xy 87.63 49.53) (xy 87.63 53.34))
     (stroke (width 0) (type default))
@@
     (effects (font (size 1.27 1.27)) (justify left bottom))
   )
+  (label "RESET" (at 181.61 100.33 0) (fields_autoplaced)
+    (effects (font (size 1.27 1.27)) (justify left bottom))
+  )
   (label "BLUE" (at 110.49 85.09 0) (fields_autoplaced)
+    (effects (font (size 1.27 1.27)) (justify left bottom))
+  )
+  (label "RESET" (at 236.22 120.65 0) (fields_autoplaced)
     (effects (font (size 1.27 1.27)) (justify left bottom))
   )
@@
     )
   )
+  (symbol (lib_id "power:GND") (at 236.22 148.59 0) (unit 1)
+    (in_bom yes) (on_board yes) (dnp no) (fields_autoplaced)
+    (property "Reference" "#PWR013" (at 236.22 154.94 0)
+      (effects (font (size 1.27 1.27)) hide)
+    )
+    (property "Value" "GND" (at 236.22 153.67 0)
+      (effects (font (size 1.27 1.27)))
+    )
+    (property "Footprint" "" (at 236.22 148.59 0)
+      (effects (font (size 1.27 1.27)) hide)
+    )
+    (property "Datasheet" "" (at 236.22 148.59 0)
+      (effects (font (size 1.27 1.27)) hide)
+    )
+    (pin "1")
+    (instances
+      (project "Akashi-18"
+        (path "/61a99dab-c882-441e-a650-f04a0666c89d"
+          (reference "#PWR013") (unit 1)
+        )
+      )
+    )
+  )
   (symbol (lib_id "Switch:SW_Omron_B3FS") (at 63.5 139.7 90) (unit 1)
     (in_bom yes) (on_board yes) (dnp no) (fields_autoplaced)
@@
         )
       )
+    )
+  )
+  (symbol (lib_id "Switch:SW_Omron_B3FS") (at 236.22 139.7 90) (unit 1)
+    (in_bom yes) (on_board yes) (dnp no) (fields_autoplaced)
+    (property "Reference" "SW4" (at 237.49 138.43 90)
+      (effects (font (size 1.27 1.27)) (justify right))
+    )
+    (property "Value" "B3FS" (at 237.49 140.97 90)
+      (effects (font (size 1.27 1.27)) (justify right))
+    )
+    (property "Footprint" "Button_Switch_THT:SW_TH_Tactile_Omron_B3F-10xx" (at 231.14 139.7 0)
+      (effects (font (size 1.27 1.27)) hide)
+    )
+    (property "Datasheet" "https://omronfs.omron.com/en_US/ecb/products/pdf/en-b3fs.pdf" (at 231.14 139.7 0)
+      (effects (font (size 1.27 1.27)) hide)
+    )
+    (pin "2")
+    (pin "1")
+    (instances
+      (project "Akashi-18"
+        (path "/61a99dab-c882-441e-a650-f04a0666c89d"
+          (reference "SW4") (unit 1)
+        )
+      )
